Commit message: [add]realsense use in gazebo

File: realsense2_description/urdf/_d435.urdf.xacro (robot description, xacro)
@@ -9,5 +9,6 @@
   <!-- Includes -->
   <xacro:include filename="$(find realsense2_description)/urdf/_materials.urdf.xacro" />
-  <xacro:macro name="sensor_d435" params="parent *origin name:=camera use_nominal_extrinsics:=false">
+  <xacro:include filename="$(find realsense2_description)/urdf/_d435_gazebo.xacro" />
+  <xacro:macro name="sensor_d435" params="name:=camera topics_ns:=camera parent  *origin ">
     <xacro:property name="M_PI" value="3.1415926535897931" />
     <!-- The following values are approximate, and the camera node
@@ -68,6 +69,4 @@
       </inertial>
     </link>
-    <!-- Use the nominal extrinsics between camera frames if the calibrated extrinsics aren't being published. e.g. running the device in simulation  -->
-    <xacro:if value="${use_nominal_extrinsics}">
       <!-- camera depth joints and links -->
       <joint name="${name}_depth_joint" type="fixed">
@@ -122,5 +121,6 @@
       </joint>
       <link name="${name}_color_optical_frame"/>
-    </xacro:if>
+    <!-- Realsense Gazebo Plugin -->
+    <xacro:gazebo_d435 camera_name="${name}" reference_link="${name}_link" topics_ns="${topics_ns}" depth_optical_frame="${name}_depth_optical_frame" color_optical_frame="${name}_color_optical_frame" infrared1_optical_frame="${name}_left_ir_optical_frame" infrared2_optical_frame="${name}_right_ir_optical_frame"/>
   </xacro:macro>
 </robot>

File: realsense2_description/urdf/test_d435_camera.urdf.xacro (robot description, xacro)
@@ -1,8 +1,7 @@
 <?xml version="1.0"?>
 <robot name="realsense2_camera" xmlns:xacro="http://ros.org/wiki/xacro">
-  <xacro:arg name="use_nominal_extrinsics" default="false"/>
   <xacro:include filename="$(find realsense2_description)/urdf/_d435.urdf.xacro" />
   <link name="base_link" />
-  <xacro:sensor_d435 parent="base_link" use_nominal_extrinsics="$(arg use_nominal_extrinsics)">
+  <xacro:sensor_d435 parent="base_link" >
     <origin xyz="0 0 0" rpy="0 0 0"/>
   </xacro:sensor_d435>
