Commit message: [fix]TF

File: realsense2_description/urdf/_d435_gazebo.xacro (robot description, xacro)
@@ -24,8 +24,9 @@
       <min_depth>0</min_depth>-->
       <sensor name="${camera_name}color" type="camera">
+        <updateRate>30</updateRate>
         <camera name="${camera_name}">
-          <horizontal_fov>${69.4*deg_to_rad}</horizontal_fov>
+          <horizontal_fov>${90*deg_to_rad}</horizontal_fov>
           <image>
-            <width>1920</width>
+            <width>3840</width>
             <height>1080</height>
             <format>RGB_INT8</format>
@@ -43,9 +44,9 @@
         <plugin name="camera_controller" filename="libgazebo_ros_camera.so">
         <alwaysOn>true</alwaysOn>
-        <updateRate>10</updateRate>
+        <updateRate>0.0</updateRate>
         <cameraName>${camera_name}</cameraName>
         <imageTopicName>image_raw</imageTopicName>
         <cameraInfoTopicName>camera_info</cameraInfoTopicName>
-        <frameName>camera_link</frameName>
+        <frameName>camera_optical_frame</frameName>
         <hackBaseline>0.07</hackBaseline>
         <distortionK1>0.0</distortionK1>
@@ -57,13 +58,16 @@
       </sensor>
       <sensor name="${camera_name}depth" type="depth">
-        <always_on>1</always_on>
-        <visualize>1</visualize>
+        <update_rate>100</update_rate>
         <camera name="${camera_name}">
-          <horizontal_fov>${91.2*deg_to_rad}</horizontal_fov>
+          <pose>0 0 0 0 0 0</pose>
+          <horizontal_fov>${90*deg_to_rad}</horizontal_fov>
           <image>
-            <width>1280</width>
-            <height>720</height>
+            <width>3840</width>
+            <height>1080</height>
             <format>B8G8R8</format>
           </image>
+          <depth_camera>
+            <output>depths</output>
+          </depth_camera>
           <clip>
             <near>0.1</near>
@@ -77,14 +81,16 @@
         </camera>
         <plugin name="${topics_ns}" filename="libgazebo_ros_openni_kinect.so">
+          <baseline>0.2</baseline>
           <alwaysOn>true</alwaysOn>
-          <updateRate>10</updateRate>
+          <updateRate>0.0</updateRate>
           <cameraName>${camera_name}_ir</cameraName>
-          <imageTopicName>/${camera_name}/depth/image_raw</imageTopicName>
-          <cameraInfoTopicName>/${camera_name}/depth/camera_info</cameraInfoTopicName>
+          <imageTopicName>/${camera_name}/color/image_raw</imageTopicName>
+          <cameraInfoTopicName>/${camera_name}/color/camera_info</cameraInfoTopicName>
           <depthImageTopicName>/${camera_name}/depth/image_raw</depthImageTopicName>
-          <depthImageInfoTopicName>/${camera_name}/depth/camera_info</depthImageInfoTopicName>
+          <depthImageCameraInfoTopicName>/${camera_name}/depth/camera_info</depthImageCameraInfoTopicName>
           <pointCloudTopicName>/${camera_name}/depth/points</pointCloudTopicName>
-          <frameName>camera_link</frameName>
-          <pointCloudCutoff>0.5</pointCloudCutoff>
+          <frameName>camera_depth_optical_frame</frameName>
+          <pointCloudCutoff>0.3</pointCloudCutoff>
+          <pointCloudCutoffMax>25.0</pointCloudCutoffMax>
           <distortionK1>0.00000001</distortionK1>
           <distortionK2>0.00000001</distortionK2>
@@ -98,5 +104,4 @@
           <hackBaseline>0</hackBaseline>
         </plugin>
-        <pose>0 0 0 0 ${radians(-90)} ${radians(90)}</pose>
       </sensor>
     </gazebo>

File: realsense2_description/urdf/test_d435_camera.urdf.xacro (robot description, xacro)
@@ -2,6 +2,6 @@
 <robot name="realsense2_camera" xmlns:xacro="http://ros.org/wiki/xacro">
   <xacro:include filename="$(find realsense2_description)/urdf/_d435.urdf.xacro" />
-  <link name="base_link" />
-  <xacro:sensor_d435 parent="base_link" >
+  <link name="world" />
+  <xacro:sensor_d435 parent="world" >
     <origin xyz="0 0 0" rpy="0 0 0"/>
   </xacro:sensor_d435>
